Commit message: feat: sync hand URDF with revo2_description v1.1.x
- Thumb abduction zero redefinition (+3 deg), MCP/PIP limits and mimic ratios
- Four-finger PIP limits 0~97 deg with per-finger mimic multipliers
- Align thumb abduction/MCP limits with mass-production version (20260818)
- Update README joint limit tables; bump package version to 1.1.1

File: urdf/revo2_left_hand.urdf (robot description, URDF)
Before this commit: robot brainco_revo2_lefthand_urdf, 22 links, 21 joints
Joints:
- joint left_index_distal_joint: limit lower=0 upper=1.63 effort=2 velocity=2.2685 -> lower=0 upper=1.69297 effort=2 velocity=2.2685; mimic joint=left_index_proximal_joint multiplier=1.155 offset=0 -> joint=left_index_proximal_joint multiplier=1.131 offset=0
- joint left_middle_distal_joint: limit lower=0 upper=1.63 effort=2 velocity=2.2685 -> lower=0 upper=1.69297 effort=2 velocity=2.2685; mimic joint=left_middle_proximal_joint multiplier=1.155 offset=0 -> joint=left_middle_proximal_joint multiplier=1.267 offset=0
- joint left_pinky_distal_joint: limit lower=0 upper=1.63 effort=2 velocity=2.2685 -> lower=0 upper=1.69297 effort=2 velocity=2.2685; mimic joint=left_pinky_proximal_joint multiplier=1.155 offset=0 -> joint=left_pinky_proximal_joint multiplier=1.271 offset=0
- joint left_ring_distal_joint: limit lower=0 upper=1.63 effort=2 velocity=2.2685 -> lower=0 upper=1.69297 effort=2 velocity=2.2685; mimic joint=left_ring_proximal_joint multiplier=1.155 offset=0 -> joint=left_ring_proximal_joint multiplier=1.252 offset=0
- joint left_thumb_distal_joint: limit lower=0 upper=1.03 effort=1.1 velocity=2.5303 -> lower=0 upper=1.15192 effort=1.1 velocity=2.5303; mimic joint=left_thumb_proximal_joint multiplier=1 offset=0 -> joint=left_thumb_proximal_joint multiplier=1.0945 offset=0; origin xyz=0 -0.052 0 rpy=0 0 0 -> xyz=0 -0.052 0 rpy=0.10472 0 0
- joint left_thumb_metacarpal_joint: limit lower=0 upper=1.57 effort=0.5 velocity=2.6175 -> lower=0 upper=1.55334 effort=0.5 velocity=2.6175; origin xyz=0.0045 -0.019 0.027825 rpy=0 0 0.16787 -> xyz=0.0045 -0.019 0.027825 rpy=0 0 0.22023
- joint left_thumb_proximal_joint: limit lower=0 upper=1.03 effort=1.1 velocity=2.5303 -> lower=0 upper=1.04720 effort=1.1 velocity=2.5303; origin xyz=0 -0.014227 0 rpy=-0.17488 0.23736 -0.16787 -> xyz=0 -0.014227 0 rpy=-0.33153 0.23736 -0.16787

File: urdf/revo2_right_hand.urdf (robot description, URDF)
Before this commit: robot brainco_revo2_righthand_urdf, 22 links, 21 joints
Joints:
- joint right_index_distal_joint: limit lower=0 upper=1.63 effort=2 velocity=2.2685 -> lower=0 upper=1.69297 effort=2 velocity=2.2685; mimic joint=right_index_proximal_joint multiplier=1.155 offset=0 -> joint=right_index_proximal_joint multiplier=1.131 offset=0
- joint right_middle_distal_joint: limit lower=0 upper=1.63 effort=2 velocity=2.2685 -> lower=0 upper=1.69297 effort=2 velocity=2.2685; mimic joint=right_middle_proximal_joint multiplier=1.155 offset=0 -> joint=right_middle_proximal_joint multiplier=1.267 offset=0
- joint right_pinky_distal_joint: limit lower=0 upper=1.63 effort=2 velocity=2.2685 -> lower=0 upper=1.69297 effort=2 velocity=2.2685; mimic joint=right_pinky_proximal_joint multiplier=1.155 offset=0 -> joint=right_pinky_proximal_joint multiplier=1.271 offset=0
- joint right_ring_distal_joint: limit lower=0 upper=1.63 effort=2 velocity=2.2685 -> lower=0 upper=1.69297 effort=2 velocity=2.2685; mimic joint=right_ring_proximal_joint multiplier=1.155 offset=0 -> joint=right_ring_proximal_joint multiplier=1.252 offset=0
- joint right_thumb_distal_joint: limit lower=0 upper=1.03 effort=1.1 velocity=2.5303 -> lower=0 upper=1.15192 effort=1.1 velocity=2.5303; mimic joint=right_thumb_proximal_joint multiplier=1 offset=0 -> joint=right_thumb_proximal_joint multiplier=1.0945 offset=0; origin xyz=0 0.052 0 rpy=0 0 0 -> xyz=0 0.052 0 rpy=-0.10472 0 0
- joint right_thumb_metacarpal_joint: limit lower=0 upper=1.57 effort=0.5 velocity=2.6175 -> lower=0 upper=1.55334 effort=0.5 velocity=2.6175; origin xyz=0.005619 0.019867 0.027825 rpy=0 0 -0.16787 -> xyz=0.005619 0.019867 0.027825 rpy=0 0 -0.22023
- joint right_thumb_proximal_joint: limit lower=0 upper=1.03 effort=1.1 velocity=2.5303 -> lower=0 upper=1.04720 effort=1.1 velocity=2.5303; origin xyz=0 0.014227 0 rpy=0.17488 0.23736 0.16787 -> xyz=0 0.014227 0 rpy=0.33153 0.23736 0.16787
